Commit message: JAKA ROS2 Package 2nd Release

File: src/jaka_a12_moveit_config/config/jaka_a12.ros2_control.xacro (robot description, xacro)
@@ -1,11 +1,16 @@
 <?xml version="1.0"?>
 <robot xmlns:xacro="http://www.ros.org/wiki/xacro">
-    <xacro:macro name="jaka_a12_ros2_control" params="name initial_positions_file">
-        <xacro:property name="initial_positions" value="${load_yaml(initial_positions_file)['initial_positions']}"/>
+    <xacro:macro name="jaka_a12_ros2_control" params="name initial_positions_file use_gazebo use_rviz_sim">
+        <xacro:property name="initial_positions" value="${xacro.load_yaml(initial_positions_file)['initial_positions']}"/>
         <ros2_control name="${name}" type="system">
             <!-- Include hardware plugin conditionally if rviz in simulation mode is enabled -->
             <hardware>
-                <!-- By default, set up controllers for simulation. This won't work on real hardware -->
-                <plugin>mock_components/GenericSystem</plugin>
+              <xacro:if value="${use_gazebo}">
+                  <!-- <plugin>gazebo_ros2_control/GazeboSystem</plugin> -->
+                  <plugin>ign_ros2_control/IgnitionSystem</plugin>
+              </xacro:if>
+              <xacro:if value="${use_rviz_sim}">
+                  <plugin>mock_components/GenericSystem</plugin>
+              </xacro:if>
             </hardware>
             <!-- Joint interfaces generated for each joint -->

File: src/jaka_a12_moveit_config/config/jaka_a12.urdf.xacro (robot description, xacro)
@@ -2,4 +2,6 @@
 <robot xmlns:xacro="http://www.ros.org/wiki/xacro" name="jaka_a12">
     <xacro:arg name="initial_positions_file" default="initial_positions.yaml" />
+    <xacro:arg name="use_gazebo" default="false"/>
+    <xacro:arg name="use_rviz_sim" default="false"/>
     <!-- Import jaka_a12 urdf file -->
     <xacro:include filename="$(find jaka_description)/urdf/jaka_a12.urdf" />
@@ -7,4 +9,4 @@
     <xacro:include filename="jaka_a12.ros2_control.xacro" />
     <!-- <xacro:jaka_a12_ros2_control name="FakeSystem" initial_positions_file="$(arg initial_positions_file)"/> -->
-    <xacro:jaka_a12_ros2_control name="jaka_a12_hardware" initial_positions_file="$(arg initial_positions_file)"/>
+    <xacro:jaka_a12_ros2_control name="jaka_a12_hardware" initial_positions_file="$(arg initial_positions_file)" use_gazebo="$(arg use_gazebo)" use_rviz_sim="$(arg use_rviz_sim)" />
 </robot>

File: src/jaka_minicobo_moveit_config/config/jaka_minicobo.ros2_control.xacro (robot description, xacro)
@@ -1,11 +1,16 @@
 <?xml version="1.0"?>
 <robot xmlns:xacro="http://www.ros.org/wiki/xacro">
-    <xacro:macro name="jaka_minicobo_ros2_control" params="name initial_positions_file">
-        <xacro:property name="initial_positions" value="${load_yaml(initial_positions_file)['initial_positions']}"/>
+    <xacro:macro name="jaka_minicobo_ros2_control" params="name initial_positions_file use_gazebo use_rviz_sim">
+        <xacro:property name="initial_positions" value="${xacro.load_yaml(initial_positions_file)['initial_positions']}"/>
         <ros2_control name="${name}" type="system">
             <!-- Include hardware plugin conditionally if rviz in simulation mode is enabled -->
             <hardware>
-                <!-- By default, set up controllers for simulation. This won't work on real hardware -->
-                <plugin>mock_components/GenericSystem</plugin>
+              <xacro:if value="${use_gazebo}">
+                  <!-- <plugin>gazebo_ros2_control/GazeboSystem</plugin> -->
+                  <plugin>ign_ros2_control/IgnitionSystem</plugin>
+              </xacro:if>
+              <xacro:if value="${use_rviz_sim}">
+                  <plugin>mock_components/GenericSystem</plugin>
+              </xacro:if>
             </hardware>
             <!-- Joint interfaces generated for each joint -->

File: src/jaka_minicobo_moveit_config/config/jaka_minicobo.urdf.xacro (robot description, xacro)
@@ -2,4 +2,6 @@
 <robot xmlns:xacro="http://www.ros.org/wiki/xacro" name="jaka_minicobo">
     <xacro:arg name="initial_positions_file" default="initial_positions.yaml" />
+    <xacro:arg name="use_gazebo" default="false"/>
+    <xacro:arg name="use_rviz_sim" default="false"/>
     <!-- Import jaka_minicobo urdf file -->
     <xacro:include filename="$(find jaka_description)/urdf/jaka_minicobo.urdf" />
@@ -7,4 +9,4 @@
     <xacro:include filename="jaka_minicobo.ros2_control.xacro" />
     <!-- <xacro:jaka_minicobo_ros2_control name="FakeSystem" initial_positions_file="$(arg initial_positions_file)"/> -->
-    <xacro:jaka_minicobo_ros2_control name="jaka_minicobo_hardware" initial_positions_file="$(arg initial_positions_file)"/>
+    <xacro:jaka_minicobo_ros2_control name="jaka_minicobo_hardware" initial_positions_file="$(arg initial_positions_file)" use_gazebo="$(arg use_gazebo)" use_rviz_sim="$(arg use_rviz_sim)" />
 </robot>

File: src/jaka_s5_moveit_config/config/jaka_s5.ros2_control.xacro (robot description, xacro)
@@ -1,11 +1,16 @@
 <?xml version="1.0"?>
 <robot xmlns:xacro="http://www.ros.org/wiki/xacro">
-    <xacro:macro name="jaka_s5_ros2_control" params="name initial_positions_file">
-        <xacro:property name="initial_positions" value="${load_yaml(initial_positions_file)['initial_positions']}"/>
+    <xacro:macro name="jaka_s5_ros2_control" params="name initial_positions_file use_gazebo use_rviz_sim">
+        <xacro:property name="initial_positions" value="${xacro.load_yaml(initial_positions_file)['initial_positions']}"/>
         <ros2_control name="${name}" type="system">
             <!-- Include hardware plugin conditionally if rviz in simulation mode is enabled -->
             <hardware>
-                <!-- By default, set up controllers for simulation. This won't work on real hardware -->
-                <plugin>mock_components/GenericSystem</plugin>
+              <xacro:if value="${use_gazebo}">
+                  <!-- <plugin>gazebo_ros2_control/GazeboSystem</plugin> -->
+                  <plugin>ign_ros2_control/IgnitionSystem</plugin>
+              </xacro:if>
+              <xacro:if value="${use_rviz_sim}">
+                  <plugin>mock_components/GenericSystem</plugin>
+              </xacro:if>
             </hardware>
             <!-- Joint interfaces generated for each joint -->

File: src/jaka_s5_moveit_config/config/jaka_s5.urdf.xacro (robot description, xacro)
@@ -2,4 +2,6 @@
 <robot xmlns:xacro="http://www.ros.org/wiki/xacro" name="jaka_s5">
     <xacro:arg name="initial_positions_file" default="initial_positions.yaml" />
+    <xacro:arg name="use_gazebo" default="false"/>
+    <xacro:arg name="use_rviz_sim" default="false"/>
     <!-- Import jaka_s5 urdf file -->
     <xacro:include filename="$(find jaka_description)/urdf/jaka_s5.urdf" />
@@ -7,4 +9,4 @@
     <xacro:include filename="jaka_s5.ros2_control.xacro" />
     <!-- <xacro:jaka_s5_ros2_control name="FakeSystem" initial_positions_file="$(arg initial_positions_file)"/> -->
-    <xacro:jaka_s5_ros2_control name="jaka_s5_hardware" initial_positions_file="$(arg initial_positions_file)"/>
+    <xacro:jaka_s5_ros2_control name="jaka_s5_hardware" initial_positions_file="$(arg initial_positions_file)" use_gazebo="$(arg use_gazebo)" use_rviz_sim="$(arg use_rviz_sim)" />
 </robot>

File: src/jaka_zu12_moveit_config/config/jaka_zu12.ros2_control.xacro (robot description, xacro)
@@ -1,11 +1,16 @@
 <?xml version="1.0"?>
 <robot xmlns:xacro="http://www.ros.org/wiki/xacro">
-    <xacro:macro name="jaka_zu12_ros2_control" params="name initial_positions_file">
-        <xacro:property name="initial_positions" value="${load_yaml(initial_positions_file)['initial_positions']}"/>
+    <xacro:macro name="jaka_zu12_ros2_control" params="name initial_positions_file use_gazebo use_rviz_sim">
+        <xacro:property name="initial_positions" value="${xacro.load_yaml(initial_positions_file)['initial_positions']}"/>
         <ros2_control name="${name}" type="system">
             <!-- Include hardware plugin conditionally if rviz in simulation mode is enabled -->
             <hardware>
-                <!-- By default, set up controllers for simulation. This won't work on real hardware -->
-                <plugin>mock_components/GenericSystem</plugin>
+              <xacro:if value="${use_gazebo}">
+                  <!-- <plugin>gazebo_ros2_control/GazeboSystem</plugin> -->
+                  <plugin>ign_ros2_control/IgnitionSystem</plugin>
+              </xacro:if>
+              <xacro:if value="${use_rviz_sim}">
+                  <plugin>mock_components/GenericSystem</plugin>
+              </xacro:if>
             </hardware>
             <!-- Joint interfaces generated for each joint -->

File: src/jaka_zu12_moveit_config/config/jaka_zu12.urdf.xacro (robot description, xacro)
@@ -2,4 +2,6 @@
 <robot xmlns:xacro="http://www.ros.org/wiki/xacro" name="jaka_zu12">
     <xacro:arg name="initial_positions_file" default="initial_positions.yaml" />
+    <xacro:arg name="use_gazebo" default="false"/>
+    <xacro:arg name="use_rviz_sim" default="false"/>
     <!-- Import jaka_zu12 urdf file -->
     <xacro:include filename="$(find jaka_description)/urdf/jaka_zu12.urdf" />
@@ -7,4 +9,4 @@
     <xacro:include filename="jaka_zu12.ros2_control.xacro" />
     <!-- <xacro:jaka_zu12_ros2_control name="FakeSystem" initial_positions_file="$(arg initial_positions_file)"/> -->
-    <xacro:jaka_zu12_ros2_control name="jaka_zu12_hardware" initial_positions_file="$(arg initial_positions_file)"/>
+    <xacro:jaka_zu12_ros2_control name="jaka_zu12_hardware" initial_positions_file="$(arg initial_positions_file)" use_gazebo="$(arg use_gazebo)" use_rviz_sim="$(arg use_rviz_sim)" />
 </robot>

File: src/jaka_zu3_moveit_config/config/jaka_zu3.ros2_control.xacro (robot description, xacro)
@@ -1,11 +1,16 @@
 <?xml version="1.0"?>
 <robot xmlns:xacro="http://www.ros.org/wiki/xacro">
-    <xacro:macro name="jaka_zu3_ros2_control" params="name initial_positions_file">
-        <xacro:property name="initial_positions" value="${load_yaml(initial_positions_file)['initial_positions']}"/>
+    <xacro:macro name="jaka_zu3_ros2_control" params="name initial_positions_file use_gazebo use_rviz_sim">
+        <xacro:property name="initial_positions" value="${xacro.load_yaml(initial_positions_file)['initial_positions']}"/>
         <ros2_control name="${name}" type="system">
             <!-- Include hardware plugin conditionally if rviz in simulation mode is enabled -->
             <hardware>
-                <!-- By default, set up controllers for simulation. This won't work on real hardware -->
-                <plugin>mock_components/GenericSystem</plugin>
+              <xacro:if value="${use_gazebo}">
+                  <!-- <plugin>gazebo_ros2_control/GazeboSystem</plugin> -->
+                  <plugin>ign_ros2_control/IgnitionSystem</plugin>
+              </xacro:if>
+              <xacro:if value="${use_rviz_sim}">
+                  <plugin>mock_components/GenericSystem</plugin>
+              </xacro:if>
             </hardware>
             <!-- Joint interfaces generated for each joint -->

File: src/jaka_zu3_moveit_config/config/jaka_zu3.urdf.xacro (robot description, xacro)
@@ -2,4 +2,6 @@
 <robot xmlns:xacro="http://www.ros.org/wiki/xacro" name="jaka_zu3">
     <xacro:arg name="initial_positions_file" default="initial_positions.yaml" />
+    <xacro:arg name="use_gazebo" default="false"/>
+    <xacro:arg name="use_rviz_sim" default="false"/>
     <!-- Import jaka_zu3 urdf file -->
     <xacro:include filename="$(find jaka_description)/urdf/jaka_zu3.urdf" />
@@ -7,4 +9,4 @@
     <xacro:include filename="jaka_zu3.ros2_control.xacro" />
     <!-- <xacro:jaka_zu3_ros2_control name="FakeSystem" initial_positions_file="$(arg initial_positions_file)"/> -->
-    <xacro:jaka_zu3_ros2_control name="jaka_zu3_hardware" initial_positions_file="$(arg initial_positions_file)"/>
+    <xacro:jaka_zu3_ros2_control name="jaka_zu3_hardware" initial_positions_file="$(arg initial_positions_file)" use_gazebo="$(arg use_gazebo)" use_rviz_sim="$(arg use_rviz_sim)" />
 </robot>

File: src/jaka_zu7_moveit_config/config/jaka_zu7.ros2_control.xacro (robot description, xacro)
@@ -1,11 +1,16 @@
 <?xml version="1.0"?>
 <robot xmlns:xacro="http://www.ros.org/wiki/xacro">
-    <xacro:macro name="jaka_zu7_ros2_control" params="name initial_positions_file">
-        <xacro:property name="initial_positions" value="${load_yaml(initial_positions_file)['initial_positions']}"/>
+    <xacro:macro name="jaka_zu7_ros2_control" params="name initial_positions_file use_gazebo use_rviz_sim">
+        <xacro:property name="initial_positions" value="${xacro.load_yaml(initial_positions_file)['initial_positions']}"/>
         <ros2_control name="${name}" type="system">
             <!-- Include hardware plugin conditionally if rviz in simulation mode is enabled -->
             <hardware>
-                <!-- By default, set up controllers for simulation. This won't work on real hardware -->
-                <plugin>mock_components/GenericSystem</plugin>
+              <xacro:if value="${use_gazebo}">
+                  <!-- <plugin>gazebo_ros2_control/GazeboSystem</plugin> -->
+                  <plugin>ign_ros2_control/IgnitionSystem</plugin>
+              </xacro:if>
+              <xacro:if value="${use_rviz_sim}">
+                  <plugin>mock_components/GenericSystem</plugin>
+              </xacro:if>
             </hardware>
             <!-- Joint interfaces generated for each joint -->

File: src/jaka_zu7_moveit_config/config/jaka_zu7.urdf.xacro (robot description, xacro)
@@ -2,4 +2,6 @@
 <robot xmlns:xacro="http://www.ros.org/wiki/xacro" name="jaka_zu7">
     <xacro:arg name="initial_positions_file" default="initial_positions.yaml" />
+    <xacro:arg name="use_gazebo" default="false"/>
+    <xacro:arg name="use_rviz_sim" default="false"/>
     <!-- Import jaka_zu7 urdf file -->
     <xacro:include filename="$(find jaka_description)/urdf/jaka_zu7.urdf" />
@@ -7,4 +9,4 @@
     <xacro:include filename="jaka_zu7.ros2_control.xacro" />
     <!-- <xacro:jaka_zu7_ros2_control name="FakeSystem" initial_positions_file="$(arg initial_positions_file)"/> -->
-    <xacro:jaka_zu7_ros2_control name="jaka_zu7_hardware" initial_positions_file="$(arg initial_positions_file)"/>
+    <xacro:jaka_zu7_ros2_control name="jaka_zu7_hardware" initial_positions_file="$(arg initial_positions_file)" use_gazebo="$(arg use_gazebo)" use_rviz_sim="$(arg use_rviz_sim)" />
 </robot>
