Commit message: fix

File: src/jaka_description/urdf/jaka_zu12_with_tool.urdf (robot description, URDF)
Before this commit: robot jaka_zu12, 9 links, 8 joints
Links:
- link connect_tool: geometry collision mesh filename=package://jaka_description/meshes/connect_tool.stl scale=0.001 0.001 0.001; visual mesh filename=package://jaka_description/meshes/connect_tool.stl scale=0.001 0.001 0.001

Commit message: Update URDF and launch script to include tool integration for Jaka ZU12 robot

File: src/jaka_description/urdf/jaka_zu12_with_tool.urdf (robot description, URDF)
Before this commit: robot jaka_zu12, 9 links, 8 joints
Links:
- link connect_tool: geometry collision mesh filename=package://jaka_description/meshes/tool/connect_tool.stl scale=0.001 0.001 0.001; visual mesh filename=package://jaka_description/meshes/tool/connect_tool.stl scale=0.001 0.001 0.001
